Commit message: fix(robotiq_description): put the Hand-E's speed and thresholds in its joint's units
- gripper_max_speed and the finger joints' velocity limit are 0.075 m/s, one finger's share of the 0.150 m/s at which the gap closes
- the topic-based stall_velocity_threshold comes from the launch per model through gripper_stall_velocity_threshold: 0.05 rad/s on the 2F models as before, 0.002 m/s on the Hand-E
- the Hand-E's topic-based hardware sends a command once 0.0005 m from the state instead of 0.02 m
- the per-model controller config tests collect without launch_ros
- README: the Hand-E's velocity and speed units, the stall threshold, and gripper_model for a custom description

Co-Authored-By: Claude Opus 5.5 <noreply@anthropic.com>

File: grippers/robotiq_description/urdf/common.ros2_control.xacro (robot description, xacro)
@@ -17,5 +17,6 @@
         gripper_max_force
         gripper_closed_position
-        gripper_profile:=''">
+        gripper_profile:=''
+        trigger_joint_command_threshold:=0.02">
         <hardware>
             <!-- Set use_dummy to true to connect to a dummy driver for testing purposes. -->
@@ -25,5 +26,5 @@
                 <param name="joint_commands_topic">${sim_joint_commands_topic}</param>
                 <param name="joint_states_topic">${sim_joint_states_topic}</param>
-                <param name="trigger_joint_command_threshold">0.02</param>
+                <param name="trigger_joint_command_threshold">${trigger_joint_command_threshold}</param>
             </xacro:if>
             <xacro:if value="${sim_gazebo}">

File: grippers/robotiq_description/urdf/hand_e.ros2_control.xacro (robot description, xacro)
@@ -35,5 +35,6 @@
                 gripper_max_force="${gripper_max_force}"
                 gripper_closed_position="${gripper_closed_position}"
-                gripper_profile="hand_e"/>
+                gripper_profile="hand_e"
+                trigger_joint_command_threshold="0.0005"/>
             <joint name="${prefix}hande_left_finger_joint">
                 <command_interface name="position" />

File: grippers/robotiq_description/urdf/robotiq_hand_e_macro.urdf.xacro (robot description, xacro)
@@ -20,5 +20,5 @@
         gripper_speed_multiplier:=1.0
         gripper_force_multiplier:=0.5
-        gripper_max_speed:=0.150
+        gripper_max_speed:=0.075
         gripper_max_force:=185.0
         gripper_closed_position:=0.025
@@ -34,4 +34,6 @@
         <xacro:property name="states_topic" value="${isaac_joint_states or ('/isaac_joint_states' if sim_isaac else sim_joint_states_topic)}"/>
         <xacro:property name="stroke" value="0.050"/>
+        <!-- One finger's top speed: the gap closes at 0.150 m/s with both moving. -->
+        <xacro:property name="finger_speed" value="0.075"/>
         <xacro:include filename="$(find robotiq_description)/urdf/hand_e.ros2_control.xacro" />
         <xacro:if value="${include_ros2_control}">
@@ -114,5 +116,5 @@
             <axis xyz="1 0 0" />
             <origin xyz="${-stroke/2} 0 0.099" rpy="0 0 0" />
-            <limit lower="0.0" upper="${stroke/2}" velocity="0.15" effort="180" />
+            <limit lower="0.0" upper="${stroke/2}" velocity="${finger_speed}" effort="180" />
         </joint>
         <joint name="${prefix}hande_right_finger_joint" type="prismatic">
@@ -121,5 +123,5 @@
             <axis xyz="-1 0 0" />
             <origin xyz="${stroke/2} 0 0.099" rpy="0 0 0" />
-            <limit lower="0.0" upper="${stroke/2}" velocity="0.15" effort="180" />
+            <limit lower="0.0" upper="${stroke/2}" velocity="${finger_speed}" effort="180" />
             <mimic joint="${prefix}hande_left_finger_joint" />
         </joint>
