Commit message: Multiple finger options

File: grippers/robotiq_description/urdf/robotiq_gripper.urdf.xacro (robot description, xacro)
@@ -16,12 +16,24 @@
     <xacro:arg name="isaac_joint_commands" default="" />
     <xacro:arg name="isaac_joint_states" default="" />
+    <xacro:arg name="finger_type" default="aluminium" />
     <!-- Import macros -->
     <xacro:include filename="$(find robotiq_description)/urdf/robotiq_$(arg gripper_model)_macro.urdf.xacro" />
     <link name="world" />
-    <xacro:robotiq_gripper name="RobotiqGripperHardwareInterface" prefix="" parent="world" use_fake_hardware="$(arg use_fake_hardware)" com_port="$(arg com_port)" baudrate="$(arg baudrate)"
-        sim_topic_based="$(arg sim_topic_based)"
-        sim_joint_commands_topic="$(arg sim_joint_commands_topic)" sim_joint_states_topic="$(arg sim_joint_states_topic)"
-        sim_isaac="$(arg sim_isaac)" isaac_joint_commands="$(arg isaac_joint_commands)" isaac_joint_states="$(arg isaac_joint_states)">
-        <origin xyz="0 0 0" rpy="0 0 0" />
-    </xacro:robotiq_gripper>
+    <xacro:if value="${'$(arg gripper_model)' == 'hand_e'}">
+        <xacro:robotiq_gripper name="RobotiqGripperHardwareInterface" prefix="" parent="world" use_fake_hardware="$(arg use_fake_hardware)" com_port="$(arg com_port)" baudrate="$(arg baudrate)"
+            sim_topic_based="$(arg sim_topic_based)"
+            sim_joint_commands_topic="$(arg sim_joint_commands_topic)" sim_joint_states_topic="$(arg sim_joint_states_topic)"
+            sim_isaac="$(arg sim_isaac)" isaac_joint_commands="$(arg isaac_joint_commands)" isaac_joint_states="$(arg isaac_joint_states)"
+            finger_type="$(arg finger_type)">
+            <origin xyz="0 0 0" rpy="0 0 0" />
+        </xacro:robotiq_gripper>
+    </xacro:if>
+    <xacro:unless value="${'$(arg gripper_model)' == 'hand_e'}">
+        <xacro:robotiq_gripper name="RobotiqGripperHardwareInterface" prefix="" parent="world" use_fake_hardware="$(arg use_fake_hardware)" com_port="$(arg com_port)" baudrate="$(arg baudrate)"
+            sim_topic_based="$(arg sim_topic_based)"
+            sim_joint_commands_topic="$(arg sim_joint_commands_topic)" sim_joint_states_topic="$(arg sim_joint_states_topic)"
+            sim_isaac="$(arg sim_isaac)" isaac_joint_commands="$(arg isaac_joint_commands)" isaac_joint_states="$(arg isaac_joint_states)">
+            <origin xyz="0 0 0" rpy="0 0 0" />
+        </xacro:robotiq_gripper>
+    </xacro:unless>
 </robot>

File: grippers/robotiq_description/urdf/robotiq_hand_e_gripper.urdf.xacro (robot description, xacro)
@@ -2,4 +2,5 @@
 <robot xmlns:xacro="http://wiki.ros.org/xacro" name="robotiq_gripper">
     <xacro:arg name="gripper_model" default="hand_e" />
+    <xacro:arg name="finger_type" default="aluminum" />
     <xacro:include filename="$(find robotiq_description)/urdf/robotiq_gripper.urdf.xacro" />
 </robot>

File: grippers/robotiq_description/urdf/robotiq_hand_e_macro.urdf.xacro (robot description, xacro)
@@ -23,5 +23,6 @@
         gripper_max_force:=185.0
         gripper_closed_position:=0.025
-        tcp_z_offset:=0.1325">
+        tcp_z_offset:=0.1325
+        finger_type:=aluminum">
         <!-- PickNik's names for the topic-based path, released in 1.1.0 and
              deprecated since 1.2.0. sim_isaac keeps its old /isaac_joint_* topic
@@ -37,4 +38,6 @@
         <xacro:property name="finger_speed" value="0.075"/>
         <xacro:include filename="$(find robotiq_description)/urdf/hand_e.ros2_control.xacro" />
+        <xacro:include filename="$(find robotiq_description)/urdf/finger_aluminum.xacro" />
+        <xacro:include filename="$(find robotiq_description)/urdf/finger_45deg.xacro" />
         <xacro:if value="${include_ros2_control}">
             <xacro:robotiq_gripper_ros2_control
@@ -95,19 +98,4 @@
                 </geometry>
             </collision>
-            <visual>
-                <origin xyz="-0.022014 0.01425 0.0015" rpy="0 0 ${pi}" />
-                <geometry>
-                    <mesh filename="package://robotiq_description/meshes/visual/hand_e/alum-finger.stl" />
-                </geometry>
-                <material name="">
-                    <color rgba="0.7 0.7 0.7 1" />
-                </material>
-            </visual>
-            <collision>
-                <origin xyz="-0.022014 0.01425 0.0015" rpy="0 0 ${pi}" />
-                <geometry>
-                    <mesh filename="package://robotiq_description/meshes/visual/hand_e/alum-finger.stl" />
-                </geometry>
-            </collision>
         </link>
         <link name="${prefix}hande_right_finger">
@@ -125,19 +113,4 @@
                 <geometry>
                     <mesh filename="package://robotiq_description/meshes/visual/hand_e/Fingerbase.stl" />
-                </geometry>
-            </collision>
-            <visual>
-                <origin xyz="0.022014 -0.01425 0.0015" rpy="0 0 0" />
-                <geometry>
-                    <mesh filename="package://robotiq_description/meshes/visual/hand_e/alum-finger.stl" />
-                </geometry>
-                <material name="">
-                    <color rgba="0.7 0.7 0.7 1" />
-                </material>
-            </visual>
-            <collision>
-                <origin xyz="0.022014 -0.01425 0.0015" rpy="0 0 0" />
-                <geometry>
-                    <mesh filename="package://robotiq_description/meshes/visual/hand_e/alum-finger.stl" />
                 </geometry>
             </collision>
@@ -160,10 +133,19 @@
             <mimic joint="${prefix}hande_left_finger_joint" />
         </joint>
-        <link name="${prefix}tcp_link" />
-        <joint name="${prefix}tcp_link_joint" type="fixed">
-            <parent link="${prefix}hand_e_base_link" />
-            <child link="${prefix}tcp_link" />
-            <origin xyz="0 0 ${tcp_z_offset}" rpy="0 0 ${-pi/2}" />
-        </joint>
+        <!-- Finger pair selection -->
+        <xacro:if value="${finger_type in ['aluminum', 'aluminium', 'alum']}">
+            <xacro:finger_aluminum prefix="${prefix}" parent_left="${prefix}hande_left_finger" parent_right="${prefix}hande_right_finger" tcp_parent="${prefix}hand_e_base_link" />
+        </xacro:if>
+        <xacro:if value="${finger_type in ['45deg', '45', 'plate']}">
+            <xacro:finger_v1 prefix="${prefix}" parent_left="${prefix}hande_left_finger" parent_right="${prefix}hande_right_finger" tcp_parent="${prefix}hand_e_base_link" />
+        </xacro:if>
+        <xacro:unless value="${finger_type in ['aluminum', 'aluminium', 'alum', '45deg', '45', 'plate']}">
+            <link name="${prefix}tcp_link" />
+            <joint name="${prefix}tcp_link_joint" type="fixed">
+                <parent link="${prefix}hand_e_base_link" />
+                <child link="${prefix}tcp_link" />
+                <origin xyz="0 0 ${tcp_z_offset}" rpy="0 0 ${-pi/2}" />
+            </joint>
+        </xacro:unless>
     </xacro:macro>
 </robot>
