Commit message: Modularized fingers (fingerbase + finger)

File: grippers/robotiq_description/urdf/robotiq_hand_e_macro.urdf.xacro (robot description, xacro)
@@ -81,6 +81,7 @@
         <link name="${prefix}hande_left_finger">
             <visual>
+                <origin xyz="0 0 0" rpy="0 0 0" />
                 <geometry>
-                    <mesh filename="package://robotiq_description/meshes/visual/hand_e/left_finger.dae" />
+                    <mesh filename="package://robotiq_description/meshes/visual/hand_e/Fingerbase.stl" />
                 </geometry>
                 <material name="">
@@ -89,13 +90,13 @@
             </visual>
             <collision>
+                <origin xyz="0 0 0" rpy="0 0 0" />
                 <geometry>
-                    <mesh filename="package://robotiq_description/meshes/collision/hand_e/left_finger.stl" />
+                    <mesh filename="package://robotiq_description/meshes/visual/hand_e/Fingerbase.stl" />
                 </geometry>
             </collision>
-        </link>
-        <link name="${prefix}hande_right_finger">
             <visual>
+                <origin xyz="-0.022014 0.01425 0.0015" rpy="0 0 ${pi}" />
                 <geometry>
-                    <mesh filename="package://robotiq_description/meshes/visual/hand_e/right_finger.dae" />
+                    <mesh filename="package://robotiq_description/meshes/visual/hand_e/alum-finger.stl" />
                 </geometry>
                 <material name="">
@@ -104,6 +105,39 @@
             </visual>
             <collision>
+                <origin xyz="-0.022014 0.01425 0.0015" rpy="0 0 ${pi}" />
                 <geometry>
-                    <mesh filename="package://robotiq_description/meshes/collision/hand_e/right_finger.stl" />
+                    <mesh filename="package://robotiq_description/meshes/visual/hand_e/alum-finger.stl" />
+                </geometry>
+            </collision>
+        </link>
+        <link name="${prefix}hande_right_finger">
+            <visual>
+                <origin xyz="0 0 0" rpy="0 0 ${pi}" />
+                <geometry>
+                    <mesh filename="package://robotiq_description/meshes/visual/hand_e/Fingerbase.stl" />
+                </geometry>
+                <material name="">
+                    <color rgba="0.7 0.7 0.7 1" />
+                </material>
+            </visual>
+            <collision>
+                <origin xyz="0 0 0" rpy="0 0 ${pi}" />
+                <geometry>
+                    <mesh filename="package://robotiq_description/meshes/visual/hand_e/Fingerbase.stl" />
+                </geometry>
+            </collision>
+            <visual>
+                <origin xyz="0.022014 -0.01425 0.0015" rpy="0 0 0" />
+                <geometry>
+                    <mesh filename="package://robotiq_description/meshes/visual/hand_e/alum-finger.stl" />
+                </geometry>
+                <material name="">
+                    <color rgba="0.7 0.7 0.7 1" />
+                </material>
+            </visual>
+            <collision>
+                <origin xyz="0.022014 -0.01425 0.0015" rpy="0 0 0" />
+                <geometry>
+                    <mesh filename="package://robotiq_description/meshes/visual/hand_e/alum-finger.stl" />
                 </geometry>
             </collision>
@@ -115,5 +149,5 @@
             <child link="${prefix}hande_left_finger" />
             <axis xyz="1 0 0" />
-            <origin xyz="${-stroke/2} 0 0.099" rpy="0 0 0" />
+            <origin xyz="0 0 0.0998" rpy="0 0 0" />
             <limit lower="0.0" upper="${stroke/2}" velocity="${finger_speed}" effort="180" />
         </joint>
@@ -122,5 +156,5 @@
             <child link="${prefix}hande_right_finger" />
             <axis xyz="-1 0 0" />
-            <origin xyz="${stroke/2} 0 0.099" rpy="0 0 0" />
+            <origin xyz="0 0 0.0998" rpy="0 0 0" />
             <limit lower="0.0" upper="${stroke/2}" velocity="${finger_speed}" effort="180" />
             <mimic joint="${prefix}hande_left_finger_joint" />

Commit message: Add inertial properties to Robotiq Hand-E fingers and adapter link in URDFs

File: grippers/robotiq_description/urdf/robotiq_hand_e_macro.urdf.xacro (robot description, xacro)
@@ -83,4 +83,9 @@
         </joint>
         <link name="${prefix}hande_left_finger">
+            <inertial>
+                <origin xyz="0 0 0.01" rpy="0 0 0" />
+                <mass value="0.038" />
+                <inertia ixx="0.00001" ixy="0" ixz="0" iyy="0.00001" iyz="0" izz="0.00001" />
+            </inertial>
             <visual>
                 <origin xyz="0 0 0" rpy="0 0 0" />
@@ -100,4 +105,9 @@
         </link>
         <link name="${prefix}hande_right_finger">
+            <inertial>
+                <origin xyz="0 0 0.01" rpy="0 0 ${pi}" />
+                <mass value="0.038" />
+                <inertia ixx="0.00001" ixy="0" ixz="0" iyy="0.00001" iyz="0" izz="0.00001" />
+            </inertial>
             <visual>
                 <origin xyz="0 0 0" rpy="0 0 ${pi}" />

File: grippers/robotiq_description/urdf/ur_to_robotiq_adapter.urdf.xacro (robot description, xacro)
@@ -33,5 +33,11 @@
       <origin xyz="0 0 0.011" rpy="0 0 0"/>
     </joint>
-    <link name="${child}"/>
+    <link name="${child}">
+      <inertial>
+        <mass value="0.001" />
+        <origin xyz="0 0 0" />
+        <inertia ixx="0.000001" ixy="0.0" ixz="0.0" iyy="0.000001" iyz="0.0" izz="0.000001" />
+      </inertial>
+    </link>
   </xacro:macro>
 </robot>
